File: the-claw-if-pizza-planet-was-broke.kicad_pcb (KiCad board)
At the start: 2 copper layers, 99.8 x 16.1 mm, 8 parts

Commit message: update with finished(?) pcb
Parts:
- removed REF** (x4): AMASS_XT30PW-F_1x02_P2.50mm_Horizontal, Connector_AMASS:AMASS_XT30PW-F_1x02_P2.50mm_Horizontal
- removed REF**: CONN-SM12B-ZPDSS-TF, the-claw:CONN-SM12B-ZPDSS-TF
- removed REF**: DIP-16_W7.62mm, Package_DIP:DIP-16_W7.62mm
- removed REF**: JST_XH_S3B-XH-A_1x03_P2.50mm_Horizontal, Connector_JST:JST_XH_S3B-XH-A_1x03_P2.50mm_Horizontal
- removed REF**: JST_XH_S4B-XH-A_1x04_P2.50mm_Horizontal, Connector_JST:JST_XH_S4B-XH-A_1x04_P2.50mm_Horizontal
- added C1: 68uF, Capacitor_THT:CP_Radial_D6.3mm_P2.50mm, F.Cu at (94.4, 71.7)
- added C2: 0.1uF, Resistor_THT:R_Axial_DIN0204_L3.6mm_D1.6mm_P2.54mm_Vertical, F.Cu at (89.1, 102.1)
- added C3: 0.1uF, Resistor_THT:R_Axial_DIN0204_L3.6mm_D1.6mm_P2.54mm_Vertical, F.Cu at (77.8, 76.1)
- added C4: 68uF, Capacitor_THT:CP_Radial_D6.3mm_P2.50mm, F.Cu at (109.8, 71.7)
- added C5: 68uF, Capacitor_THT:CP_Radial_D6.3mm_P2.50mm, F.Cu at (66.0, 71.7)
- added C6: 68uF, Capacitor_THT:CP_Radial_D6.3mm_P2.50mm, F.Cu at (65.8, 97.3)
- added D1: D_Small, Diode_THT:D_DO-35_SOD27_P7.62mm_Horizontal, F.Cu at (115.6, 83.6)
- added J1: Conn_01x02, Connector_AMASS:AMASS_XT30PW-M_1x02_P2.50mm_Horizontal, F.Cu at (81.7, 66.0)
- added J10: Conn_01x04, Connector_JST:JST_XH_S4B-XH-A-1_1x04_P2.50mm_Horizontal, F.Cu at (65.8, 103.7)
- added J11: Conn_01x04_Socket, the-claw:DB125-2.54-4P, F.Cu at (138.2, 70.8)
- added J12: Conn_01x04_Socket, the-claw:DB125-2.54-4P, F.Cu at (132.0, 70.8)
- added J13: Conn_03x03_Odd_Even, the-claw:PinHeader_3x03_P2.54mm_Vertical, F.Cu at (116.8, 124.0)
- added J14: Conn_01x02, Connector_AMASS:AMASS_XT60PW-F_1x02_P7.20mm_Horizontal, F.Cu at (62.4, 136.4)
- added J15: Conn_01x02, Connector_AMASS:AMASS_XT60PW-F_1x02_P7.20mm_Horizontal, F.Cu at (78.8, 136.4)
- added J2: Conn_01x02, Connector_AMASS:AMASS_XT30PW-M_1x02_P2.50mm_Horizontal, F.Cu at (96.0, 66.0)
- added J3: Conn_01x02, Connector_AMASS:AMASS_XT30PW-M_1x02_P2.50mm_Horizontal, F.Cu at (67.3, 66.0)
- added J4: Conn_01x02, Connector_AMASS:AMASS_XT30PW-M_1x02_P2.50mm_Horizontal, F.Cu at (110.2, 66.0)
- added J5: Conn_01x04, Connector_JST:JST_XH_S4B-XH-A-1_1x04_P2.50mm_Horizontal, F.Cu at (136.2, 60.5)
- added J6: Conn_02x06_Odd_Even, the-claw:CONN-SM12B-ZPDSS-TF, F.Cu at (148.2, 58.2)
- added J7: Conn_01x03, Connector_JST:JST_XH_S3B-XH-A_1x03_P2.50mm_Horizontal, F.Cu at (122.8, 62.1)
- added J8: Conn_01x03_Socket, the-claw:DB125-2.54-3P, F.Cu at (125.6, 69.5)
- added J9: Conn_01x02, Connector_PinHeader_2.54mm:PinHeader_1x02_P2.54mm_Vertical, F.Cu at (118.6, 89.2)
- added Q1: MS50N, Package_TO_SOT_SMD:TO-252-2, F.Cu at (137.9, 83.7)
- added Q2: MS50N, Package_TO_SOT_SMD:TO-252-2, F.Cu at (120.3, 78.5)
- added Q3: MS50N, Package_TO_SOT_SMD:TO-252-2, F.Cu at (130.9, 83.7)
- added Q4: MS50N, Package_TO_SOT_SMD:TO-252-2, F.Cu at (84.5, 126.6)
- added Q5: BSS84, Package_TO_SOT_SMD:SOT-23, F.Cu at (65.9, 127.3)
- added R1: 8.2k, Resistor_THT:R_Axial_DIN0207_L6.3mm_D2.5mm_P10.16mm_Horizontal, F.Cu at (91.3, 86.5)
- added R10: 10k, Resistor_THT:R_Axial_DIN0207_L6.3mm_D2.5mm_P10.16mm_Horizontal, F.Cu at (62.7, 132.4)
- added R11: 10k, Resistor_THT:R_Axial_DIN0207_L6.3mm_D2.5mm_P10.16mm_Horizontal, F.Cu at (72.5, 129.0)
- added R12: 10k, Resistor_THT:R_Axial_DIN0207_L6.3mm_D2.5mm_P10.16mm_Horizontal, F.Cu at (68.9, 115.2)
- added R2: 470, Resistor_THT:R_Axial_DIN0207_L6.3mm_D2.5mm_P10.16mm_Horizontal, F.Cu at (88.3, 73.1)
- added R3: 1k, Resistor_THT:R_Axial_DIN0207_L6.3mm_D2.5mm_P10.16mm_Horizontal, F.Cu at (85.3, 73.1)
- added R4: 10k, Resistor_THT:R_Axial_DIN0207_L6.3mm_D2.5mm_P10.16mm_Horizontal, F.Cu at (105.2, 97.1)
- added R5: 3.3k, Resistor_THT:R_Axial_DIN0204_L3.6mm_D1.6mm_P5.08mm_Horizontal, F.Cu at (102.6, 104.7)
- added R6: 10k, Resistor_THT:R_Axial_DIN0207_L6.3mm_D2.5mm_P10.16mm_Horizontal, F.Cu at (129.8, 118.9)
- added R7: 10k, Resistor_THT:R_Axial_DIN0207_L6.3mm_D2.5mm_P10.16mm_Horizontal, F.Cu at (87.8, 109.8)
- added R8: 10k, Resistor_THT:R_Axial_DIN0207_L6.3mm_D2.5mm_P10.16mm_Horizontal, F.Cu at (87.8, 112.8)
- added R9: 10k, Resistor_THT:R_Axial_DIN0207_L6.3mm_D2.5mm_P10.16mm_Horizontal, F.Cu at (59.7, 122.2)
- added U1: COS29752, Package_TO_SOT_SMD:TO-263-5_TabPin3, F.Cu at (75.5, 83.6)
- added U2: COS29752, Package_TO_SOT_SMD:TO-263-5_TabPin3, F.Cu at (95.8, 98.2)
- added U3: PCF8574AP, Package_DIP:DIP-16_W7.62mm, F.Cu at (119.7, 124.0)
- added U4: 74LV1T08GW, Package_TO_SOT_SMD:SOT-353_SC-70-5, F.Cu at (115.2, 96.3)
Routing:
- net +3V3: track 0.00 -> 163.6 mm, vias 0 -> 1
- net /I2C_SCL: track 0.00 -> 160.9 mm, vias 0 -> 1
- net /I2C_SDA: track 0.00 -> 154.2 mm, vias 0 -> 1
- net +24V: track 0.00 -> 153.5 mm
- net +5V: track 0.00 -> 130.5 mm, vias 0 -> 1
- net +12V: track 0.00 -> 94.1 mm, vias 0 -> 1
- net /VACUUM_ENABLE: track 0.00 -> 54.7 mm
- net /SOLENOID_ENABLE: track 0.00 -> 49.2 mm
- net /LASER_PWM_3V3: track 0.00 -> 43.7 mm
- net /LASER_PWM: track 0.00 -> 36.9 mm
- net /VACUUM_GND: track 0.00 -> 23.6 mm
- net /SOLENOID_GND: track 0.00 -> 22.8 mm
- net GND: track 0.00 -> 15.8 mm, vias 0 -> 1
- net /LASER_GND: track 0.00 -> 15.2 mm
- net Net-(U1-ADJ): track 0.00 -> 14.3 mm
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- added copper zone on F.Cu, net +12V
- added copper zone on F.Cu, net +5V
- added copper zone on B.Cu, net /BED_24V
- added copper zone on F.Cu, net /BED_GND
- added copper zone on F.Cu, net GND
- added copper zone on F.Cu, net Net-(J15-Pin_2)
Other:
- board size 99.8 x 16.1 mm -> 99.8 x 99.8 mm
- board text added: "The Claw"
- board text added: "bed control"

Commit message: fix a bunch of stuff
Parts:
- added H1: MountingHole, MountingHole:MountingHole_4.3mm_M4, F.Cu at (151.4, 124.5)
- added H2: MountingHole, MountingHole:MountingHole_4.3mm_M4, F.Cu at (132.8, 146.6)
- added J16: Conn_01x03, Connector_JST:JST_XH_B3B-XH-A_1x03_P2.50mm_Vertical, F.Cu at (146.0, 79.0)
- added Q6: AO3400A, Package_TO_SOT_SMD:SOT-23, F.Cu at (143.1, 88.9)
- added U5: TMP100, Package_TO_SOT_SMD:SOT-23-6, F.Cu at (72.6, 114.0)
- J14: footprint Connector_AMASS:AMASS_XT60PW-F_1x02_P7.20mm_Horizontal -> Connector_JST:JST_XH_S2B-XH-A-1_1x02_P2.50mm_Horizontal
- J3: footprint Connector_AMASS:AMASS_XT30PW-M_1x02_P2.50mm_Horizontal -> Connector_AMASS:AMASS_XT60PW-F_1x02_P7.20mm_Horizontal
- moved R7 20.4 mm to (69.4, 118.7)
- moved R8 18.6 mm to (69.4, 115.7)
- moved C3 12.7 mm to (75.5, 88.6)
- moved Q5 10.5 mm to (65.5, 137.8)
- moved R12 10.1 mm to (65.3, 124.7)
- moved C2 9.56 mm to (95.2, 109.4), turned to 180 degrees
- moved J14 7.94 mm to (60.8, 144.2), turned to 0 degrees
- moved U1 7.93 mm to (80.3, 77.3)
- moved R11 7.19 mm to (68.3, 134.8)
- moved R10 6.31 mm to (62.3, 138.7)
- moved R9 6.31 mm to (59.3, 128.5)
- moved Q4 5.00 mm to (87.8, 130.3), turned to 180 degrees
- moved J11 4.00 mm to (142.2, 70.4)
- moved R6 3.75 mm to (129.8, 122.7)
- moved J3 3.15 mm to (69.5, 68.3)
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Connections:
- J14 pad 2: /BED_GND -> /BED_CONTROL
- J15 pad 1: /BED_24V -> +24V
- Q4 pad 3: /BED_GND -> GND
- R10 pad 1: /BED_GND -> /BED_CONTROL
- R11 pad 1: /BED_GND -> GND
- U3 pad 7: unconnected-(U3-P3-Pad7) -> /FAN_ENABLE
Routing:
- net /FAN_ENABLE: track 0.00 -> 62.8 mm, vias 0 -> 1
- net +24V: track 153.5 -> 212.1 mm
- net +3V3: track 163.6 -> 192.9 mm, vias 1 -> 4
- net +12V: track 94.1 -> 121.5 mm, vias 1 -> 0
- net /I2C_SCL: track 160.9 -> 182.0 mm, vias 1 -> 5
- net Net-(Q4-G): track 14.3 -> 32.4 mm, vias 0 -> 1
- net /LASER_PWM_3V3: track 43.7 -> 55.8 mm, vias 0 -> 1
- net /SOLENOID_ENABLE: track 49.2 -> 56.3 mm, vias 0 -> 1
- net Net-(Q5-G): track 8.89 -> 15.9 mm
- net Net-(U1-ADJ): track 14.3 -> 7.46 mm
- net /LASER_POWER: track 6.02 -> 12.5 mm
- net /BED_CONTROL: track 0.00 -> 5.87 mm
- net /VACUUM_ENABLE: track 54.7 -> 60.5 mm, vias 0 -> 1
- net GND: track 15.8 -> 10.2 mm, vias 1 -> 0
- net /BED_24V: track 7.90 -> 13.2 mm
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- added copper zone on B.Cu, net +24V
- added copper zone on B.Cu, net +5V
- removed copper zone on F.Cu, net +12V
- removed copper zone on B.Cu, net /BED_24V
- removed copper zone on F.Cu, net /BED_GND
Other:
- board text added: "24V in 24V out 12V out 5V out Laser: PWR/GND/PWM PNP: Vacuum PWR/GND Solenoid PWR/GND I/O (see schematic)"
- board text added: "5.8A max fan power draw Everything else may draw up to 7.5A, it's only a matter of whether the connectors can handle it (voltage drop will likely occur) XH rated 3A ZPD rated 2A per pin XT30 rated 15A XT60 rated 30A"
- board text removed: "bed control"
