File: the-claw-if-pizza-planet-was-broke.kicad_pcb (KiCad board)
At the start: 2 copper layers, 99.8 x 99.8 mm, 48 parts, among them J1 Conn_01x02, J10 Conn_01x04, J11 Conn_01x04_Socket, J12 Conn_01x04_Socket, J13 Conn_03x03_Odd_Even, J14 Conn_01x02, J15 Conn_01x02, J16 Conn_01x03, J2 Conn_01x02, J3 Conn_01x02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

Commit message: give XT30 hrt
Parts:
- J1, J2, J4: footprint Connector_AMASS:AMASS_XT30PW-M_1x02_P2.50mm_Horizontal -> Connector_AMASS:AMASS_XT30PW-F_1x02_P2.50mm_Horizontal
- moved J2 5.13 mm to (93.1, 67.0)
- moved J4 5.13 mm to (107.4, 67.0)
- moved J1 5.13 mm to (78.8, 67.0)
- moved C1 1.56 mm to (96.6, 73.2), turned to 0 degrees
- moved C4 0.95 mm to (109.8, 72.6)
Connections:
- J1 pad 1: +24V -> GND
- J1 pad 2: GND -> +24V
- J2 pad 1: +12V -> GND
- J2 pad 2: GND -> +12V
- J4 pad 1: +5V -> GND
- J4 pad 2: GND -> +5V
Routing:
- net +12V: track 121.5 -> 163.5 mm
- net +5V: track 126.0 -> 130.3 mm

Commit message: update w/ XT60 + silkscreen improvement
Parts:
- J3: footprint Connector_AMASS:AMASS_XT60PW-F_1x02_P7.20mm_Horizontal -> Connector_AMASS:AMASS_XT60PW-M_1x02_P7.20mm_Horizontal
- moved J3 7.27 mm to (62.3, 69.3)
- moved C3 4.37 mm to (79.9, 88.6)
- moved C5 2.54 mm to (64.5, 74.2), turned to 0 degrees
Routing:
- net +24V: track 212.1 -> 264.8 mm, vias 0 -> 12
- net Net-(J15-Pin_2): track 0.00 -> 6.25 mm
- net Net-(Q4-G): track 32.4 -> 30.8 mm
- added copper zone on B.Cu, net GND
- removed copper zone on B.Cu, net +24V
Other:
- board text added: "**BED**"
- board text added: "24V 12V 5V PWR"
- board text added: "24V 12V PWR"
- board text added: "24V GND"
- board text added: "3.3V GND SCL SDA"
- board text added: "PWM GND PWR"
- board text added: "PWR 5V 12V 24V"
- board text added: "SOL GND SOL PWR VAC GND VAC PWR"
