File: the-claw-if-pizza-planet-was-broke.kicad_sch (KiCad schematic)
At the start: 43 parts, among them J1 Conn_01x02, J10 Conn_01x04, J11 Conn_01x04_Socket, J12 Conn_01x04_Socket, J13 Conn_03x03_Odd_Even, J14 Conn_01x02, J15 Conn_01x02, J2 Conn_01x02, J3 Conn_01x02, J4 Conn_01x02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

Commit message: update with finished(?) pcb
Parts:
- removed Q1, Q2, Q3, Q4: Q_NMOS, symbol Device:Q_NMOS
- removed Q5: Q_PMOS, symbol Device:Q_PMOS
- added Q1, Q2, Q3, Q4: MS50N, Package_TO_SOT_SMD:TO-252-2, symbol the-claw:MS50N
- added Q5: BSS84, Package_TO_SOT_SMD:SOT-23, symbol Transistor_FET:BSS84
- C1, C4, C5, C6: footprint (none) -> Capacitor_THT:CP_Radial_D6.3mm_P2.50mm
- C2, C3: footprint (none) -> Resistor_THT:R_Axial_DIN0204_L3.6mm_D1.6mm_P2.54mm_Vertical
- D1: footprint (none) -> Diode_THT:D_DO-35_SOD27_P7.62mm_Horizontal
- J10, J5: footprint (none) -> Connector_JST:JST_XH_S4B-XH-A-1_1x04_P2.50mm_Horizontal
- J11, J12: footprint (none) -> the-claw:DB125-2.54-4P
- J14, J15: footprint Connector_AMASS:AMASS_XT30PW-M_1x02_P2.50mm_Horizontal -> Connector_AMASS:AMASS_XT60PW-F_1x02_P7.20mm_Horizontal
- J6: footprint (none) -> the-claw:CONN-SM12B-ZPDSS-TF
- J7: footprint (none) -> Connector_JST:JST_XH_S3B-XH-A_1x03_P2.50mm_Horizontal
- J8: footprint (none) -> the-claw:DB125-2.54-3P
- J9: footprint (none) -> Connector_PinHeader_2.54mm:PinHeader_1x02_P2.54mm_Vertical
- R1, R10, R11, R12, R2, R3, R4, R7, R8, R9: footprint (none) -> Resistor_THT:R_Axial_DIN0207_L6.3mm_D2.5mm_P10.16mm_Horizontal
- R5: renamed from R6; footprint (none) -> Resistor_THT:R_Axial_DIN0204_L3.6mm_D1.6mm_P5.08mm_Horizontal
- R6: renamed from R5; footprint (none) -> Resistor_THT:R_Axial_DIN0207_L6.3mm_D2.5mm_P10.16mm_Horizontal
- U1, U2: footprint Package_TO_SOT_SMD:TO-263-5_TabPin6 -> Package_TO_SOT_SMD:TO-263-5_TabPin3
Connections:
- net BED_24V: now also Q5.3 (D)
- net BED_GND: now also Q4.3 (S)
- net GND: now also Q1.3 (S), Q2.3 (S), Q3.3 (S)
- net LASER_GND: now also Q2.2 (D)
- net LASER_PWM: no longer U3.4 (P0)
- net LASER_PWM_3V3: now also U3.4 (P0)
- net SOLENOID_ENABLE: now also U3.5 (P1), Q3.1 (G); no longer U3.6 (P2)
- net SOLENOID_GND: now also Q3.2 (D)
- net VACUUM_ENABLE: now also U3.6 (P2), Q1.1 (G); no longer U3.5 (P1)
- net VACUUM_GND: now also Q1.2 (D)
- net at R11.2, R12.1: now also Q4.1 (G)
- net at J15.2 (Pin_2): now also Q4.2 (D)
- net at D1.1 (K), J9.2 (Pin_2): now also Q2.1 (G)
- net at R10.2, R9.1: now also Q5.1 (G)
- net at R12.2: now also Q5.2 (S)

Commit message: fix a bunch of stuff
Parts:
- added H1, H2: MountingHole, MountingHole:MountingHole_4.3mm_M4, symbol Mechanical:MountingHole
- added J16: Conn_01x03, Connector_JST:JST_XH_B3B-XH-A_1x03_P2.50mm_Vertical, symbol Connector_Generic:Conn_01x03
- added Q6: AO3400A, Package_TO_SOT_SMD:SOT-23, symbol Transistor_FET:AO3400A
- added U5: TMP100, Package_TO_SOT_SMD:SOT-23-6, symbol Sensor_Temperature:TMP100
- J14: footprint Connector_AMASS:AMASS_XT60PW-F_1x02_P7.20mm_Horizontal -> Connector_JST:JST_XH_S2B-XH-A-1_1x02_P2.50mm_Horizontal
- J3: footprint Connector_AMASS:AMASS_XT30PW-M_1x02_P2.50mm_Horizontal -> Connector_AMASS:AMASS_XT60PW-F_1x02_P7.20mm_Horizontal
Connections:
- net +12V: now also J16.2 (Pin_2)
- net +24V: now also J15.1 (Pin_1), J16.1 (Pin_1)
- net +3V3: now also U5.4 (V+)
- net BED_24V: no longer J15.1 (Pin_1)
- net GND: now also Q4.3 (S), R11.1, Q6.2 (S), U5.2 (GND), U5.3 (ADD1), U5.5 (ADD0)
- net I2C_SCL: now also U5.1 (SCL)
- net I2C_SDA: now also U5.6 (SDA)
- net FAN_ENABLE: now reaches U3.7 (P3)
- net FAN_ENABLE: now also Q6.1 (G)
- net BED_GND renamed BED_CONTROL
- net BED_CONTROL: no longer Q4.3 (S), R11.1
- new net: J16.3 (Pin_3), Q6.3 (D)
Other:
- note added: "WARNING this is designed for 7.5A going to any output (except fans - 5.8A max) however, XH is only rated for 3A, and ZPD for 2A. use above that current at your own risk"
- note added: "add 5v if possible maybe?"
- note added: "could just use normal 24V here but 1) trying to make sure no meaningful power goes through that 2) most viable connector is JST XH 2P anyways and this should be simpler"
- note removed: "WARNING if possible, this will be designed for 7.5A going to any output. however, XH is only rated for 3A, and ZPD for 2A. use above that current at your own risk"
- moved on the sheet: J15, Q4, Q5, R10, R11, R12, R9

Commit message: give XT30 hrt
Parts:
- J1, J2, J4: footprint Connector_AMASS:AMASS_XT30PW-M_1x02_P2.50mm_Horizontal -> Connector_AMASS:AMASS_XT30PW-F_1x02_P2.50mm_Horizontal
Connections:
- net +12V: now also J2.2 (Pin_2); no longer J2.1 (Pin_1)
- net +24V: now also J1.2 (Pin_2); no longer J1.1 (Pin_1)
- net +5V: now also J4.2 (Pin_2); no longer J4.1 (Pin_1)
- net GND: now also J1.1 (Pin_1), J2.1 (Pin_1), J4.1 (Pin_1); no longer J1.2 (Pin_2), J2.2 (Pin_2), J4.2 (Pin_2)
Other:
- moved on the sheet: J1, J2, J4

Commit message: update w/ XT60 + silkscreen improvement
Parts:
- J3: footprint Connector_AMASS:AMASS_XT60PW-F_1x02_P7.20mm_Horizontal -> Connector_AMASS:AMASS_XT60PW-M_1x02_P7.20mm_Horizontal
